File: Hardware/Prototype/STM32 Driver v1/STM32 Driver v1.sch (KiCad schematic (older format))
At the start: 40 parts, among them J1 DBG, J2 5V PWR, J3 HUB75, J4 LEDs, J5 SPI, J6 UART, SW1 RST, U1 AP2112K-3.3, U2 STM32F411RETx, U3 74HC245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

Commit message: STM32F411RE Board Bringup complete
Parts:
- U1: symbol Regulator_Linear:AP2112K-3.3 -> STM32-Driver-v1-rescue:AP2112K-3.3-Regulator_Linear
Changed lines of the file:
@@
 $EndComp
 $Comp
-L Regulator_Linear:AP2112K-3.3 U1
+L STM32-Driver-v1-rescue:AP2112K-3.3-Regulator_Linear U1
 U 1 1 5F99E634
 P 3700 1200
