File: Hardware/Prototype/STM32 Driver v1/STM32 Driver v1.kicad_pcb (KiCad board)
At the start: 4 copper layers, 68.3 x 34.3 mm, 43 parts, among them J1 DBG, J2 5V PWR, J3 HUB75, J4 LEDs, J5 SPI, J6 UART, SW1 SW_SPST, U1 AP2112K-3.3, U2 STM32F411RETx, U3 74HC245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

Commit message: VSCode compilation of ES32 and STM32 code
Connections:
- net ~OE renamed ~{OE}
- net ~RESET renamed ~{RESET}
Routing:
- net SWCLK: track 28.5 -> 5.73 mm
- net GND: track 52.7 -> 47.0 mm, vias 33 -> 30
- net +3V3: track 30.7 -> 28.6 mm, vias 10 -> 9
- net ~{RESET}: track 43.7 -> 42.1 mm
- net SWDIO: track 21.3 -> 20.9 mm, vias 2 -> 3
Other:
- net class Default removed
